Commit message: xacro package name

File: phx_odometry/urdf/quadrotor.urdf.xacro (robot description, xacro)
@@ -10,5 +10,5 @@
         <origin xyz="0 0 0" rpy="0 0 0" />
         <geometry>
-          <mesh filename="package://phoenix_odometry/meshes/quadrotor_base.dae"/>
+          <mesh filename="package://phx_odometry/meshes/quadrotor_base.dae"/>
         </geometry>
       </visual>
@@ -16,5 +16,5 @@
         <origin xyz="0 0 0" rpy="0 0 0" />
         <geometry>
-          <mesh filename="package://phoenix_odometry/meshes/quadrotor_base.stl"/>
+          <mesh filename="package://phx_odometry/meshes/quadrotor_base.stl"/>
         </geometry>
       </collision>

Commit message: set urdf file to baselink, publish initial heading to hector and reset

File: phx_odometry/urdf/quadrotor.urdf.xacro (robot description, xacro)
@@ -1,7 +1,7 @@
 <?xml version="1.0"?>
 <robot xmlns:xacro="http://ros.org/wiki/xacro" name="phoenix">
-    <link name="drone">
+    <link name="base_link">
       <inertial>
-        <mass value="1.477" />
+        <mass value="2.5" />
         <origin xyz="0 0 0" />
         <inertia ixx="0.01152" ixy="0.0" ixz="0.0" iyy="0.01152" iyz="0.0" izz="0.0218" />
